File: GettingToBlinky/GettingToBlinky.kicad_pcb (KiCad board)
At the start: 2 copper layers, 6 parts, among them U1 7555

Commit message: autorouting
Parts:
- C1: footprint Capacitors_SMD:C_0805_HandSoldering -> Capacitors_THT:C_Disc_D7.5mm_W2.5mm_P5.00mm
- D1: footprint LEDs:LED_1206_HandSoldering -> LEDs:LED_D1.8mm_W1.8mm_H2.4mm_Horizontal_O1.27mm_Z8.2mm
- R1, R2, R3: footprint Resistors_SMD:R_0805_HandSoldering -> Resistors_THT:R_Axial_DIN0309_L9.0mm_D3.2mm_P2.54mm_Vertical
- U1: footprint Housings_SOIC:HTSOP-8-1EP_3.9x4.9mm_Pitch1.27mm -> Housings_SOIC:HTSOP-8-1EP_3.9x4.9mm_Pitch1.27mm_ThermalVias
- moved R3 35.5 mm to (134.1, 98.6), turned to 270 degrees
- moved D1 28.3 mm to (138.7, 111.3), turned to 180 degrees
- moved U1 15.4 mm to (143.8, 98.0), turned to 0 degrees
- moved C1 9.06 mm to (158.5, 95.5), turned to 270 degrees
- moved R1 5.98 mm to (143.3, 110.7), turned to 0 degrees
- moved R2 5.29 mm to (151.4, 106.2), turned to 0 degrees
Routing:
- net GND: track 17.1 -> 0.00 mm
- net Net-(C1-Pad1): track 15.5 -> 0.00 mm
- net Net-(D1-Pad2): track 14.3 -> 0.00 mm
- net Net-(R1-Pad2): track 10.5 -> 0.00 mm
- net Net-(R3-Pad1): track 10.3 -> 0.00 mm
- net /VDD: track 9.50 -> 0.00 mm
