File: GettingToBlinky/GettingToBlinky.sch (KiCad schematic (older format))
At the start: 7 parts, among them U1 7555

Commit message: schema
Parts:
- C1: footprint Capacitors_SMD:C_0805_HandSoldering -> Capacitors_THT:C_Disc_D7.5mm_W2.5mm_P5.00mm
- D1: footprint LEDs:LED_1206_HandSoldering -> LEDs:LED_D1.8mm_W1.8mm_H2.4mm_Horizontal_O1.27mm_Z8.2mm
- R1, R2, R3: footprint Resistors_SMD:R_0805_HandSoldering -> Resistors_THT:R_Axial_DIN0309_L9.0mm_D3.2mm_P2.54mm_Vertical
- U1: footprint Housings_SOIC:HTSOP-8-1EP_3.9x4.9mm_Pitch1.27mm -> Housings_SOIC:HTSOP-8-1EP_3.9x4.9mm_Pitch1.27mm_ThermalVias
Changed lines of the file:
@@
 F 0 "U1" H 4500 1825 60  0000 C CNN
 F 1 "7555" H 4100 2500 60  0000 C CNN
-F 2 "Housings_SOIC:HTSOP-8-1EP_3.9x4.9mm_Pitch1.27mm" H 4450 2875 60  0001 C CNN
+F 2 "Housings_SOIC:HTSOP-8-1EP_3.9x4.9mm_Pitch1.27mm_ThermalVias" H 4450 2875 60  0001 C CNN
 F 3 "" H 4450 2875 60  0001 C CNN
 	1    4050 2500
@@
 F 0 "R1" V 2730 1900 50  0000 C CNN
 F 1 "1K" V 2650 1900 50  0000 C CNN
-F 2 "Resistors_SMD:R_0805_HandSoldering" V 2580 1900 50  0001 C CNN
+F 2 "Resistors_THT:R_Axial_DIN0309_L9.0mm_D3.2mm_P2.54mm_Vertical" V 2580 1900 50  0001 C CNN
 F 3 "" H 2650 1900 50  0001 C CNN
 	1    2650 1900
@@
 F 0 "R2" V 2730 2450 50  0000 C CNN
 F 1 "470K" V 2650 2450 50  0000 C CNN
-F 2 "Resistors_SMD:R_0805_HandSoldering" V 2580 2450 50  0001 C CNN
+F 2 "Resistors_THT:R_Axial_DIN0309_L9.0mm_D3.2mm_P2.54mm_Vertical" V 2580 2450 50  0001 C CNN
 F 3 "" H 2650 2450 50  0001 C CNN
 	1    2650 2450
@@
 F 0 "C1" H 2675 3300 50  0000 L CNN
 F 1 "1mF" H 2675 3100 50  0000 L CNN
-F 2 "Capacitors_SMD:C_0805_HandSoldering" H 2688 3050 50  0001 C CNN
+F 2 "Capacitors_THT:C_Disc_D7.5mm_W2.5mm_P5.00mm" H 2688 3050 50  0001 C CNN
 F 3 "" H 2650 3200 50  0001 C CNN
 	1    2650 3200
@@
 F 0 "D1" H 4950 3000 50  0000 C CNN
 F 1 "LED" H 4950 2800 50  0000 C CNN
-F 2 "LEDs:LED_1206_HandSoldering" H 4950 2900 50  0001 C CNN
+F 2 "LEDs:LED_D1.8mm_W1.8mm_H2.4mm_Horizontal_O1.27mm_Z8.2mm" H 4950 2900 50  0001 C CNN
 F 3 "" H 4950 2900 50  0001 C CNN
 	1    4950 2900
@@
 F 0 "R3" V 5030 2500 50  0000 C CNN
 F 1 "1K" V 4950 2500 50  0000 C CNN
-F 2 "Resistors_SMD:R_0805_HandSoldering" V 4880 2500 50  0001 C CNN
+F 2 "Resistors_THT:R_Axial_DIN0309_L9.0mm_D3.2mm_P2.54mm_Vertical" V 4880 2500 50  0001 C CNN
 F 3 "" H 4950 2500 50  0001 C CNN
 	1    4950 2500
